Commit message: slam added and working but diffdrive control BT due to which map is very distorted

File: src/drive/urdf/drive_gazebo.urdf (robot description, URDF)
Before this commit: robot drive, 16 links, 15 joints
Joints:
- joint lidar_joint: origin xyz=0.25 -0.38 0.52 rpy=0 0 0 -> xyz=0.25 -0.38 0.80 rpy=0 0 0

Commit message: fixed the control joy a bit, j is forward and else acco

File: src/drive/urdf/drive_gazebo.urdf (robot description, URDF)
Before this commit: robot drive, 16 links, 15 joints
Joints:
- joint joint_wheel_1: axis 0.99619 -0.014024 -0.08602 -> -0.99619 0.014024 0.08602
- joint joint_wheel_2: axis 0.99619 -0.014024 -0.08602 -> -0.99619 0.014024 0.08602
- joint joint_wheel_3: axis 0.99619 -0.014024 -0.08602 -> -0.99619 0.014024 0.08602
- joint joint_wheel_4: axis 0.99619 -0.014024 -0.08602 -> -0.99619 0.014024 0.08602
- joint joint_wheel_5: axis 0.99619 -0.014024 -0.08602 -> -0.99619 0.014024 0.08602
- joint joint_wheel_6: axis 0.99619 -0.014024 -0.08602 -> -0.99619 0.014024 0.08602
